Commit message: Recongifured for V2 and URDF

File: urdf/robaka_v2.xacro (robot description, xacro)
@@ -7,7 +7,7 @@
   <xacro:property name="base_wheel_gap" value="0.02"/>
   <xacro:property name="wheel_separation" value="0.31"/>
-  <xacro:property name="wheel_joint_offset" value="0.105"/>
+  <xacro:property name="wheel_joint_offset" value="-0.107"/>
   <xacro:property name="caster_wheel_radius" value="0.0375"/>
-  <xacro:property name="caster_wheel_joint_offset" value="-0.08"/>
+  <xacro:property name="caster_wheel_joint_offset" value="0.12"/>
   <xacro:include filename="$(find robaka)/urdf/robaka_v2_gazebo_plugins.xacro"/>
   <material name="blue">
@@ -126,3 +126,30 @@
     <origin xyz="${caster_wheel_joint_offset} 0 -${0.06+caster_wheel_radius}" rpy="0 0 0"/>
   </joint>
+  <joint name="imu_joint" type="fixed">
+    <parent link="base_link" />
+    <child link="imu" />
+    <origin xyz="0.16 -0.065 0.035" rpy="0 0 0" />
+  </joint>
+  <link name="imu" />
+  <joint name="lidar_joint" type="fixed">
+    <parent link="base_link" />
+    <child link="lidar" />
+    <origin xyz="0.0 0.0 0.12" rpy="0 0 3.14159" />
+  </joint>
+  <link name="lidar">
+    <visual>
+      <material name="blue" />
+      <origin xyz="0 0 0" rpy="0 0 0"/>
+      <geometry>
+        <cylinder radius="0.032" length="0.02"/>
+      </geometry>
+    </visual>
+  </link>
+  <joint name="camera_joint" type="fixed">
+    <origin xyz="0.185 0 0.07" rpy="0 0 0" />
+    <parent link="base_link" />
+    <child link="camera" />
+  </joint>
+  <link name="camera" type="fixed">
+  </link>
 </robot>

Commit message: RTABMAP WIP

File: urdf/robaka_v2.xacro (robot description, xacro)
@@ -10,4 +10,5 @@
   <xacro:property name="caster_wheel_radius" value="0.0375"/>
   <xacro:property name="caster_wheel_joint_offset" value="0.12"/>
+  <xacro:property name="realsense_height" value="1.05"/>
   <xacro:include filename="$(find robaka)/urdf/robaka_v2_gazebo_plugins.xacro"/>
   <material name="blue">
@@ -146,4 +147,5 @@
     </visual>
   </link>
+  <!--
   <joint name="camera_joint" type="fixed">
     <origin xyz="0.185 0 0.07" rpy="0 0 0" />
@@ -153,3 +155,18 @@
   <link name="camera" type="fixed">
   </link>
+  -->
+  <joint name="realsense_joint" type="fixed">
+    <parent link="base_link" />
+    <child link="camera_link" />
+    <origin xyz="0.185 0 ${realsense_height}" rpy="0 0 0" />
+  </joint>
+  <link name="camera_link" type="fixed">
+     <visual>
+      <material name="blue" />
+      <origin xyz="0 0 0" rpy="0 0 0"/>
+      <geometry>
+        <cylinder radius="0.015" length="0.08"/>
+      </geometry>
+    </visual>
+  </link>
 </robot>

Commit message: Fixed warnings, added laser_filters to remove robot elements from the scan

File: urdf/robaka_v2.xacro (robot description, xacro)
@@ -37,4 +37,5 @@
     </inertial>
   </xacro:macro>
+  <link name="dummy"/>
   <link name="base_footprint">
     <xacro:box_inertia m="8" w="0.001" h="0.001" d="0.001"/>
@@ -47,4 +48,8 @@
     </visual>
   </link>
+  <joint name="dummy_joint" type="fixed">
+     <parent link="dummy"/>
+     <child link="base_footprint"/>
+   </joint>
   <link name="base_link">
     <xacro:box_inertia m="1" w="${base_len}" h="${base_width}" d="0.01"/>
@@ -149,7 +154,7 @@
     <origin xyz="0.185 0 0.07" rpy="0 0 0" />
     <parent link="base_link" />
-    <child link="camera" />
+    <child link="camera_link" />
   </joint>
-  <link name="camera" type="fixed">
+  <link name="camera_link" type="fixed">
   </link>
 </robot>

Commit message: Fixed URDF

File: urdf/robaka_v2.xacro (robot description, xacro)
@@ -51,5 +51,5 @@
      <parent link="dummy"/>
      <child link="base_footprint"/>
-   </joint>
+     </joint>
   <link name="base_link">
     <xacro:box_inertia m="1" w="${base_len}" h="${base_width}" d="0.01"/>
@@ -94,5 +94,5 @@
       <xacro:cylinder_inertia m="10" r="${wheel_radius}" h="0.02"/>
     </link>
-    <joint name="${prefix}_wheel_joint" type="continuous">
+    <joint name="${prefix}_wheel" type="continuous">
       <axis xyz="0 1 0" rpy="0 0 0" />
       <parent link="base_link"/>

Commit message: Fix URDF

File: urdf/robaka_v2.xacro (robot description, xacro)
@@ -90,5 +90,5 @@
       <xacro:cylinder_inertia m="10" r="${wheel_radius}" h="0.02"/>
     </link>
-    <joint name="${prefix}_wheel_joint" type="continuous">
+    <joint name="${prefix}_wheel" type="continuous">
       <axis xyz="0 1 0" rpy="0 0 0" />
       <parent link="base_link"/>

Commit message: Added simple AR tag follower

File: urdf/robaka_v2.xacro (robot description, xacro)
@@ -152,5 +152,5 @@
   </link>
   <joint name="camera_joint" type="fixed">
-    <origin xyz="0.185 0 0.07" rpy="0 0 0" />
+    <origin xyz="0.185 0 0.07" rpy="0 0 3.14159" />
     <parent link="base_link" />
     <child link="camera_link" />

Commit message: Progress with move_base and AR tracking

File: urdf/robaka_v2.xacro (robot description, xacro)
@@ -2,5 +2,5 @@
 <robot xmlns:xacro="http://www.ros.org/wiki/xacro" name="robaka_v2">
   <xacro:property name="base_width" value="0.3"/>
-  <xacro:property name="base_len" value="0.4"/>
+  <xacro:property name="base_len" value="0.46"/>
   <xacro:property name="base_height" value="0.12"/>
   <xacro:property name="wheel_radius" value="0.085"/>
@@ -51,5 +51,5 @@
      <parent link="dummy"/>
      <child link="base_footprint"/>
-     </joint>
+  </joint>
   <link name="base_link">
     <xacro:box_inertia m="1" w="${base_len}" h="${base_width}" d="0.01"/>
@@ -152,9 +152,15 @@
   </link>
   <joint name="camera_joint" type="fixed">
-    <origin xyz="0.185 0 0.07" rpy="0 0 3.14159" />
+    <origin xyz="0.270 0 0.10" rpy="0 0 0" />
     <parent link="base_link" />
     <child link="camera_link" />
   </joint>
   <link name="camera_link" type="fixed">
+    <visual>
+      <material name="lightgray"/>
+      <geometry>
+        <box size="0.025 0.09 0.025"/>
+      </geometry>
+    </visual>
   </link>
 </robot>
